Commit message: whooops, forgot to save some files

File: description/lidar.xacro (robot description, xacro)
@@ -3,9 +3,6 @@
   <!-- properties -->
   <xacro:property name="wl_ldr_base" value="0.0556"/>
-<<<<<<< HEAD
-=======
   <xacro:property name="h_offset" value="0.103"/>
   <xacro:property name="l_offset" value="-0.07"/>
->>>>>>> 8dfc5c0d7a9da5742bd655b1c45715c0cc800bc5
   <xacro:property name="h_ldr_base" value="0.0231"/>
   <xacro:property name="r_ldr_top" value="${wl_ldr_base/2 - 0.001}"/>
@@ -14,18 +11,10 @@
   <xacro:property name="m_ldr_top" value="0.1"/>
   <xacro:property name="h_ldr_trans" value="0.0298"/>
-<<<<<<< HEAD
-  <xacro:property name="material" value="blue"/>
-=======
   <xacro:property name="color" value="blue"/>
->>>>>>> 8dfc5c0d7a9da5742bd655b1c45715c0cc800bc5
   <!-- joints and links -->
   <joint name="laser_base_joint" type="fixed">
     <parent link="chassis"/>
     <child link="laser_base_link"/>
-<<<<<<< HEAD
-    <origin xyz="${l_chs/3} 0 ${h_chs/2}" rpy="0 0 0"/>
-=======
     <origin xyz="${l_offset} 0 ${h_chs/2 + h_offset}" rpy="0 0 0"/>
->>>>>>> 8dfc5c0d7a9da5742bd655b1c45715c0cc800bc5
   </joint>
   <!-- radar base is the box -->
@@ -36,9 +25,5 @@
         <box size="${wl_ldr_base} ${wl_ldr_base} ${h_ldr_base}"/>
       </geometry>
-<<<<<<< HEAD
-      <material name="${material}"/>
-=======
       <material name="${color}"/>
->>>>>>> 8dfc5c0d7a9da5742bd655b1c45715c0cc800bc5
     </visual>
     <collision>
@@ -65,9 +50,5 @@
         <cylinder radius="${r_ldr_top}" length="${h_ldr_top}"/>
       </geometry>
-<<<<<<< HEAD
-      <material name="black"/>
-=======
       <material name="${color}"/>
->>>>>>> 8dfc5c0d7a9da5742bd655b1c45715c0cc800bc5
     </visual>
     <collision>
@@ -81,46 +62,7 @@
     <parent link="laser_base_link"/>
     <child link="laser_transducer_frame"/>
-<<<<<<< HEAD
-    <origin xyz="0.0 0.0 ${h_ldr_trans}" rpy="0 0.0 ${pi/2}"/>
-=======
     <origin xyz="0.0 0.0 ${h_ldr_trans}" rpy="0 0 3.1416"/>  <!-- 180 degrees because lidar is oriented wrong -->
->>>>>>> 8dfc5c0d7a9da5742bd655b1c45715c0cc800bc5
   </joint>
   <link name="laser_transducer_frame">
   </link>
-<<<<<<< HEAD
-  <!-- ================================================== -->
-  <!-- ============  GAZEBO STUFF  ====================== -->
-  <!-- ================================================== -->
-  <gazebo reference="laser_transducer_frame">
-    <sensor name="lidar_c3" type="ray">
-      <pose>0 0 0 0 0 0</pose>
-      <visualize>true</visualize>
-      <update_rate>10</update_rate>
-      <ray>
-        <scan>
-          <horizontal>
-            <samples>360</samples>
-            <resolution>1</resolution>
-            <min_angle>-3.14</min_angle>
-            <max_angle>3.14</max_angle>
-          </horizontal>
-        </scan>
-        <range>
-          <min>0.05</min>
-          <max>12.0</max>
-          <resolution>0.015</resolution>
-        </range>
-      </ray>
-      <plugin name="lidar_controller" filename="libgazebo_ros_ray_sensor.so">
-        <ros>
-          <argument>~/out:=scan</argument>
-        </ros>
-        <output_type>sensor_msgs/LaserScan</output_type>
-        <frame_name>laser_transducer_frame</frame_name>
-      </plugin>
-    </sensor>
-  </gazebo>
-=======
->>>>>>> 8dfc5c0d7a9da5742bd655b1c45715c0cc800bc5
 </robot>

File: description/robot.urdf.xacro (robot description, xacro)
@@ -2,12 +2,6 @@
 <robot xmlns:xacro="http://www.ros.org/wiki/xacro"  name="robot">
     <xacro:include filename="robot_core.xacro" />
-<<<<<<< HEAD
-    <xacro:include filename="lidar.xacro"/>
-    <xacro:include filename="ros2_control.xacro" />
-    <!-- <xacro:include filename="gz_control.xacro" /> -->
-=======
     <xacro:include filename="lidar.xacro" />
     <xacro:include filename="camera.xacro" />
     <xacro:include filename="ros2_control.xacro" />
->>>>>>> 8dfc5c0d7a9da5742bd655b1c45715c0cc800bc5
 </robot>

File: description/robot_core.xacro (robot description, xacro)
@@ -24,9 +24,5 @@
     <!-- SAXIBOT PROPERTIES -->
     <!-- wheels -->
-<<<<<<< HEAD
-    <xacro:property name="d_whl" value="0.144"/>
-=======
     <xacro:property name="d_whl" value="0.142"/>
->>>>>>> 8dfc5c0d7a9da5742bd655b1c45715c0cc800bc5
     <xacro:property name="r_whl" value="${d_whl/2}"/>
     <xacro:property name="l_whl" value="0.04"/>
@@ -34,11 +30,4 @@
     <!-- chassis -->
     <xacro:property name="l_chs" value="0.4"/>  <!-- length is the depth (x) -->
-<<<<<<< HEAD
-    <xacro:property name="w_chs" value="0.4"/>  <!-- width is the front-face width (y)-->
-    <xacro:property name="h_chs" value="0.2"/>  <!-- height is the height (z) -->
-    <xacro:property name="dx_whl" value="${l_chs/3}"/>  <!-- offset of wheels wrt center box -->
-    <xacro:property name="dz_whl" value="${h_chs/2}"/>  <!-- offset of wheels wrt center box -->
-    <xacro:property name="dy_whl" value="${l_whl/2 + w_chs/2 + 0.003}"/> <!-- 3 mm buffer-->
-=======
     <xacro:property name="w_chs" value="0.3"/>  <!-- width is the front-face width (y)-->
     <xacro:property name="h_chs" value="0.15"/>  <!-- height is the height (z) -->
@@ -46,5 +35,4 @@
     <xacro:property name="dz_whl" value="${h_chs/2}"/>  <!-- offset of wheels wrt center box -->
     <xacro:property name="dy_whl" value="${l_whl/2 + w_chs/2 + 0.004}"/> <!-- 3 mm buffer-->
->>>>>>> 8dfc5c0d7a9da5742bd655b1c45715c0cc800bc5
     <xacro:property name="xyz_chs" value="${l_chs} ${w_chs} ${h_chs}"/>
     <xacro:property name="m_chs" value="3.0"/>  <!-- estimated weight (uniform for now) -->

File: description/ros2_control.xacro (robot description, xacro)
@@ -5,7 +5,4 @@
     <!-- HARDWARE INTERFACE for CM -->
     <hardware>
-<<<<<<< HEAD
-      <plugin>gz_ros2_control/GazeboSimSystem</plugin>
-=======
       <plugin>diffdrive_arduino/DiffDriveArduino</plugin>
       <param name="left_wheel_name">left_wheel_joint</param>
@@ -17,5 +14,4 @@
       <param name="enc_counts_per_rev">4480</param>
       <param name="timeout">1000</param>
->>>>>>> 8dfc5c0d7a9da5742bd655b1c45715c0cc800bc5
     </hardware>
     <!-- joints -->
